File: mandela.kicad_pcb (KiCad board)
At the start: 2 copper layers, 64 x 54.4 mm, 3 parts

Commit message: Update files
Parts:
- added G***: LOGO, LOGO, F.Cu at (219.0, 54.0)
- added G***: LOGO, LOGO, F.Cu at (181.0, 54.0)
- added G***: LOGO, LOGO, B.Cu at (200.6, 45.6)
- added R2: R, no_silk:R_Axial_DIN0207_L6.3mm_D2.5mm_P7.62mm_Horizontal, F.Cu at (196.4, 48.0)
- added RV1: R_Potentiometer, no_silk:Potentiometer_Vishay_T73YP_Vertical, F.Cu at (202.5, 42.5)
- D2: footprint LED_THT:LED_D5.0mm -> no_silk:LED_D5.0mm
Connections:
- D2 pad 2: Net-(BT1-+) -> Net-(D2-A)
Routing:
- net Net-(BT1-+): track 50.5 -> 38.5 mm
- net Net-(R2-Pad1): track 0.00 -> 9.55 mm
- net Net-(D2-A): track 0.00 -> 7.41 mm
- net unconnected-(RV1-Pad3): track 0.00 -> 5.31 mm
- net Net-(BT1--): track 47.7 -> 52.4 mm
